Commit message: new camera link

File: src/bugger/urdf/issac_seven.urdf (robot description, URDF)
Before this commit: robot issac_seven, 13 links, 12 joints
Links:
- added link depth_camera_optical_frame
Joints:
- added joint depth_camera_optical_joint: type fixed, parent depth_camera, child depth_camera_optical_frame, origin xyz=0 0 0 rpy=-1.5708 0 -1.5708

Commit message: revert camera

File: src/bugger/urdf/issac_seven.urdf (robot description, URDF)
Before this commit: robot issac_seven, 14 links, 13 joints
Links:
- removed link depth_camera_optical_frame
Joints:
- removed joint depth_camera_optical_joint

Commit message: depth camera axes change

File: src/bugger/urdf/issac_seven.urdf (robot description, URDF)
Before this commit: robot issac_seven, 13 links, 12 joints
Joints:
- joint dcamera: origin xyz=0 0 0 rpy=0 0 0 -> xyz=0 0 0 rpy=-1.5708 0 -1.5708

Commit message: Yaw changes in urdf

File: src/bugger/urdf/issac_seven.urdf (robot description, URDF)
Before this commit: robot issac_seven, 13 links, 12 joints
Joints:
- joint dcamera: origin xyz=0 0 0 rpy=-1.5708 0 -1.5708 -> xyz=0 0 0 rpy=-1.5708 0 0
